Commit message: update dg, add marker

File: src/omron_moma/robot_description/urdf/MoMa_TM12.urdf (robot description, URDF)
Before this commit: robot AMR_Platform, 20 links, 19 joints
Links:
- removed link base
- removed link flange_link
- removed link link_0
- removed link link_1
- removed link link_2
- removed link link_3
- removed link link_4
- removed link link_5
- removed link link_6
- removed link main_body
- removed link tool0
- added link amr_main_body, mass 4.07; collision mesh filename=package://amr_visualisation/meshes/AMR_Platform.STL; visual mesh filename=package://amr_visualisation/meshes/AMR_Platform.STL
- added link flange
- added link tm_base
- added link tm_link_0, mass 1.0; collision mesh filename=package://tm_models/meshes/tm12_1300/collision/tm12_base_c.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; visual mesh filename=package://tm_models/meshes/tm12_1300/visual/tm12_base.stl
- added link tm_link_1, mass 4.5; collision mesh filename=package://tm_models/meshes/tm12_1300/collision/tm_750w_01_c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; visual mesh filename=package://tm_models/meshes/tm12_1300/visual/tm_750w_01.stl
- added link tm_link_2, mass 11.0; collision mesh filename=package://tm_models/meshes/tm12_1300/collision/tm12_arm1_c.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; visual mesh filename=package://tm_models/meshes/tm12_1300/visual/tm12_arm1.stl
- added link tm_link_3, mass 2.5; collision mesh filename=package://tm_models/meshes/tm12_1300/collision/tm12_arm2_c.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; visual mesh filename=package://tm_models/meshes/tm12_1300/visual/tm12_arm2.stl
- added link tm_link_4, mass 1.45; collision mesh filename=package://tm_models/meshes/tm12_1300/collision/tm_100w_01_c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; visual mesh filename=package://tm_models/meshes/tm12_1300/visual/tm_100w_01.stl
- added link tm_link_5, mass 1.45; collision mesh filename=package://tm_models/meshes/tm12_1300/collision/tm_100w_02_c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; visual mesh filename=package://tm_models/meshes/tm12_1300/visual/tm_100w_02.stl
- added link tm_link_6, mass 0.4; collision mesh filename=package://tm_models/meshes/tm12_1300/collision/tm_ee_c.stl; visual mesh filename=package://tm_models/meshes/tm12_1300/visual/tm_ee.stl
Joints:
- removed joint base-base_link
- removed joint flange_link-tool0
- removed joint main_body_to_base
- added joint amr_main_body_to_base: type fixed, parent base_link, child amr_main_body, origin xyz=0 0 0.085
- added joint tm_base_link: type fixed, parent tm_base, child tm_link_0, origin xyz=0 0 0 rpy=1.5708 0 0
- joint chassis_connector: parent main_body -> amr_main_body
- joint flange_fixed_joint: child flange_link -> flange; parent link_6 -> tm_link_6
- joint joint_1: child link_1 -> tm_link_1; parent link_0 -> tm_link_0
- joint joint_2: child link_2 -> tm_link_2; parent link_1 -> tm_link_1
- joint joint_3: child link_3 -> tm_link_3; parent link_2 -> tm_link_2
- joint joint_4: child link_4 -> tm_link_4; parent link_3 -> tm_link_3
- joint joint_5: child link_5 -> tm_link_5; parent link_4 -> tm_link_4
- joint joint_6: child link_6 -> tm_link_6; parent link_5 -> tm_link_5
- joint joint_EOAT: parent flange_link -> flange
- joint left_back_small_wheel_joint: parent main_body -> amr_main_body
- joint left_front_small_wheel_joint: parent main_body -> amr_main_body
- joint left_wheel_joint: parent main_body -> amr_main_body
- joint right_back_small_wheel_joint: parent main_body -> amr_main_body
- joint right_front_small_wheel_joint: parent main_body -> amr_main_body
- joint right_wheel_joint: parent main_body -> amr_main_body
- joint tm_connector: child link_0 -> tm_base; origin xyz=-0.25 0 0.75 rpy=1.57 0 1.57 -> xyz=-0.25 0 0.73 rpy=0 0 1.5708
