Commit message: add tm12 model urdf to moma

File: src/omron_moma/robot_description/urdf/MoMa.urdf (robot description, URDF)
Before this commit: robot AMR_Platform, 18 links, 18 joints
Joints:
- joint tm_connector: origin xyz=-0.25 0 0.7 rpy=0 0 1.57 -> xyz=-0.25 0 0.75 rpy=0 0 1.57

Commit message: Update MoMa to use new features from AMR and TM

File: src/omron_moma/robot_description/urdf/MoMa.urdf (robot description, URDF)
Before this commit: robot AMR_Platform, 18 links, 18 joints
Links:
- removed link link_0
- added link tm_base; collision mesh filename=package://tmr_description/meshes/tm5-900/collision/tm5_base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; visual mesh filename=package://tmr_description/meshes/tm5-900/visual/tm5_base.obj
Joints:
- joint base_fixed_joint: child link_0 -> tm_base
- joint joint_1: parent link_0 -> tm_base
- joint tm_connector: child link_0 -> tm_base

Commit message: Remove ugly AMR platform

File: src/omron_moma/robot_description/urdf/MoMa.urdf (robot description, URDF)
Before this commit: robot AMR_Platform, 18 links, 18 joints
Links:
- removed link left_back_small_wheel
- removed link left_front_small_wheel
- removed link left_wheel
- removed link right_back_small_wheel
- removed link right_front_small_wheel
- removed link right_wheel
- link main_body: geometry collision mesh filename=package://amr_visualisation/meshes/LD90.obj; visual mesh filename=package://amr_visualisation/meshes/LD90.obj
Joints:
- removed joint left_back_small_wheel_joint
- removed joint left_front_small_wheel_joint
- removed joint left_wheel_joint
- removed joint right_back_small_wheel_joint
- removed joint right_front_small_wheel_joint
- removed joint right_wheel_joint
- joint main_body_to_base: origin xyz=0 0 0.085 -> xyz=0 0 0
